File: modular-processing-board/mcu.kicad_sch (KiCad schematic)
At the start: 51 parts, among them J201 Conn_ARM_SWD_TagConnect_TC2030, J202 Conn_02x06_Odd_Even, SW201 SW_Push, SW602 SW_Push, U201 STM32H723ZGTx, U202 SRV05-4, Y1201 25MHz

Commit message: minor changes in BOM and DNP-components
Parts:
- TP201, TP202: now left out of the parts list

Commit message: changed footprints (next) try uploading to jlcpcb for manufacturing, change crystal if required for economic assembly
Parts:
- R1201: footprint Resistor_SMD:R_0402_1005Metric_Pad0.72x0.64mm_HandSolder -> Resistor_SMD:R_0603_1608Metric; LPN C17168 -> C21189; MPN 0402WGF0000TCE -> 0603WAF0000T5E
- R203, R207, R217, R218: footprint Resistor_SMD:R_0805_2012Metric_Pad1.20x1.40mm_HandSolder -> Resistor_SMD:R_0603_1608Metric; LPN C17477 -> C21189; MPN 0805W8F0000T5E -> 0603WAF0000T5E

Commit message: processing hw submitted
Parts:
- removed Y1201: 25MHz, Crystal:Crystal_SMD_3225-4Pin_3.2x2.5mm, symbol Device:Crystal_GND24_Small
- added Y201: 8MHz, Crystal:Crystal_SMD_5032-2Pin_5.0x3.2mm, symbol Device:Crystal_Small
- C1227, C201: value 4.7pF -> 20pF; LPN C1569 -> C1554; MPN 0402CG4R7C500NT -> 0402CG200J500NT
Connections:
- net HSE_OUT: now also Y201.2
- net at C201.2, R1201.1: now also Y201.1

Commit message: changed testpoints
Parts:
- TP201, TP202: footprint iw-misc:TestPoint_Pad_D0.5mm -> Connector_PinSocket_1.27mm:PinSocket_1x01_P1.27mm_Vertical
