File: modular-processing-board/power.kicad_sch (KiCad schematic)
At the start: 11 parts, among them J701 Conn_02x02_Odd_Even, U701 AMS1117-3.3

Commit message: changed footprints (next) try uploading to jlcpcb for manufacturing, change crystal if required for economic assembly
Parts:
- C701, C702, C703: footprint Capacitor_SMD:C_0805_2012Metric -> Capacitor_SMD:C_0603_1608Metric; LPN C45783 -> C59461; MPN CL21A226MAQNNNE -> CL10A226MQ8NRNC
Changed lines of the file:
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@@
 		)
 		(property "Value" "22uF"
-			(at 109.982 78.232 0)
+			(at 109.982 57.404 0)
 			(effects
 				(font
@@
 			)
 		)
-		(property "Footprint" "Capacitor_SMD:C_0805_2012Metric"
+		(property "Footprint" "Capacitor_SMD:C_0603_1608Metric"
 			(at 113.03 80.01 0)
 			(effects
@@
 			)
 		)
-		(property "LPN" "C45783"
+		(property "LPN" "C59461"
 			(at 113.03 80.01 0)
 			(effects
@@
 			)
 		)
-		(property "MPN" "CL21A226MAQNNNE"
+		(property "MPN" "CL10A226MQ8NRNC"
 			(at 113.03 80.01 0)
 			(effects
@@
 			)
 		)
-		(property "Footprint" "Capacitor_SMD:C_0805_2012Metric"
+		(property "Footprint" "Capacitor_SMD:C_0603_1608Metric"
 			(at 107.95 80.01 0)
 			(effects
@@
 			)
 		)
-		(property "LPN" "C45783"
+		(property "LPN" "C59461"
 			(at 107.95 80.01 0)
 			(effects
@@
 			)
 		)
-		(property "MPN" "CL21A226MAQNNNE"
+		(property "MPN" "CL10A226MQ8NRNC"
 			(at 107.95 80.01 0)
 			(effects
@@
 			)
 		)
-		(property "Footprint" "Capacitor_SMD:C_0805_2012Metric"
+		(property "Footprint" "Capacitor_SMD:C_0603_1608Metric"
 			(at 118.11 80.01 0)
 			(effects
@@
 			)
 		)
-		(property "LPN" "C45783"
+		(property "LPN" "C59461"
 			(at 118.11 80.01 0)
 			(effects
@@
 			)
 		)
-		(property "MPN" "CL21A226MAQNNNE"
+		(property "MPN" "CL10A226MQ8NRNC"
 			(at 118.11 80.01 0)
 			(effects

Commit message: changed testpoints
Parts:
- TP701: footprint iw-misc:TestPoint_Pad_D0.5mm -> Connector_PinSocket_1.27mm:PinSocket_1x01_P1.27mm_Vertical
Changed lines of the file:
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@@
 			)
 		)
-		(property "Footprint" "iw-misc:TestPoint_Pad_D0.5mm"
+		(property "Footprint" "Connector_PinSocket_1.27mm:PinSocket_1x01_P1.27mm_Vertical"
 			(at 53.34 43.18 0)
 			(effects
